File: Main/Main.kicad_pcb (KiCad board)
At the start: 2 copper layers, 18 parts, among them J1 AdvancedConnector1, J2 Fires, J3 Conn_01x08_Socket, M1 ServoHandL, M2 ServoHandR, M3 ServoRotateFry, M4 ServoFixFry, M5 MotorLT, M6 MotorLB, M7 MotorRT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

Commit message: センサー関係忘れてた
Parts:
- added J4: Conn_01x02_Socket, Connector_PinSocket_2.54mm:PinSocket_1x02_P2.54mm_Vertical, F.Cu at (58.4, 86.4)
- added J5: Conn_01x02_Socket, Connector_PinSocket_2.54mm:PinSocket_1x02_P2.54mm_Vertical, F.Cu at (58.4, 91.4)
- added REF**: MountingHole_3.2mm_M3, MountingHole:MountingHole_3.2mm_M3, F.Cu at (59.7, 109.2)
- added REF**: MountingHole_3.2mm_M3, MountingHole:MountingHole_3.2mm_M3, F.Cu at (59.7, 40.6)
- added REF**: MountingHole_3.2mm_M3, MountingHole:MountingHole_3.2mm_M3, F.Cu at (113.0, 109.2)
- added REF**: MountingHole_3.2mm_M3, MountingHole:MountingHole_3.2mm_M3, F.Cu at (113.0, 40.6)
- BT1, J2, M5, M6, M7, M8: footprint Connector_PinHeader_2.54mm:PinHeader_1x02_P2.54mm_Vertical -> Connector_PinSocket_2.54mm:PinSocket_1x02_P2.54mm_Vertical
- M4: footprint Connector_PinSocket_2.54mm:PinSocket_1x03_P2.54mm_Vertical -> Connector_PinHeader_2.54mm:PinHeader_1x03_P2.54mm_Vertical
- moved LS1 92.0 mm to (96.5, 111.8), turned to -90 degrees
- moved J2 90.4 mm to (104.1, 111.8), turned to 90 degrees
- moved Q1 71.7 mm to (88.9, 102.9), turned to 90 degrees
- moved U2 55.8 mm to (74.9, 102.9), turned to -90 degrees
- moved BT1 26.7 mm to (118.1, 101.6), turned to 180 degrees
- moved J1 9.16 mm to (58.4, 48.3)
- moved J3 5.08 mm to (58.4, 63.5)
- moved M8 2.84 mm to (118.1, 53.3)
- moved M6 2.84 mm to (118.1, 81.3)
- moved U3 2.54 mm to (104.1, 91.4)
- moved U4 2.54 mm to (104.1, 63.5)
- moved U1 2.54 mm to (66.0, 38.1)
- moved M5 1.27 mm to (118.1, 91.4)
- moved M7 1.27 mm to (118.1, 63.5)
Connections:
- U1 pad 19: unconnected-(U1-GPIO17/U1TXD/ADC2_CH6/DAC_1-Pad19) -> GPIO17
Routing:
- net GND: track 0.00 -> 182.3 mm
- net VCC: track 0.00 -> 119.0 mm
- net Fire: track 0.00 -> 53.9 mm
- net GND1: track 0.00 -> 46.1 mm
- net VCCQ: track 0.00 -> 40.9 mm
- net DF_TX: track 0.00 -> 40.8 mm, vias 0 -> 1
- net DF_RX: track 0.00 -> 39.3 mm, vias 0 -> 1
- net Net-(U2-SPK2): track 0.00 -> 35.3 mm
- net Net-(U2-SPK1): track 0.00 -> 33.5 mm
- net Net-(J2-Pin_1): track 0.00 -> 18.9 mm
- net PWM_RotateFry: track 0.00 -> 14.4 mm
- net PWM_HandR: track 0.00 -> 14.4 mm
- net PWM_HandL: track 0.00 -> 14.4 mm
- net PWM_FixFry: track 0.00 -> 14.4 mm
- net L_BI_P: track 0.00 -> 10.8 mm
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Other:
- board outline added: 65.3 x 78.6 mm

Commit message: 出力を追加
Parts:
- removed J4, J5: Conn_01x02_Socket, Connector_PinSocket_2.54mm:PinSocket_1x02_P2.54mm_Vertical
- added J6: Conn_01x08_Socket, Connector_PinSocket_2.54mm:PinSocket_1x08_P2.54mm_Vertical, F.Cu at (58.4, 83.8)
- J1: value AdvancedConnector1 -> AdvancedConnector; footprint Connector_PinSocket_2.54mm:PinSocket_1x06_P2.54mm_Vertical -> Connector_PinSocket_2.54mm:PinSocket_1x08_P2.54mm_Vertical
- J3: value Conn_01x08_Socket -> Conn_01x04_Socket; footprint Connector_PinSocket_2.54mm:PinSocket_1x08_P2.54mm_Vertical -> Connector_PinSocket_2.54mm:PinSocket_1x04_P2.54mm_Vertical
- moved J3 5.08 mm to (58.4, 68.6)
- moved REF** 4.84 mm to (117.5, 111.1)
- moved REF** 4.44 mm to (117.5, 40.6)
- moved REF** 1.91 mm to (59.7, 111.1)
Connections:
- J3 pad 3: Net-(J3-Pin_3) -> VCC
- J3 pad 4: Net-(J3-Pin_4) -> GND
- U1 pad 11: Net-(J3-Pin_1) -> Net-(J1-Pin_7)
- U1 pad 12: Net-(J3-Pin_2) -> Net-(J1-Pin_8)
- U1 pad 13: Net-(J3-Pin_3) -> Net-(J3-Pin_1)
- U1 pad 14: Net-(J3-Pin_4) -> Net-(J3-Pin_2)
- U1 pad 15: Net-(J3-Pin_5) -> GPIO13
- U1 pad 16: Net-(J3-Pin_6) -> GPIO14
Routing:
- net VCC: track 119.0 -> 159.5 mm, vias 0 -> 2
- net GND: track 182.3 -> 202.2 mm
- net GPIO14: track 0.00 -> 14.1 mm
- net GPIO13: track 0.00 -> 13.3 mm
- net Net-(J3-Pin_6): track 7.62 -> 0.00 mm
- net Net-(J3-Pin_5): track 7.62 -> 0.00 mm
- net Net-(J3-Pin_4): track 7.62 -> 0.00 mm
- net Net-(J3-Pin_3): track 7.62 -> 0.00 mm
- net Net-(J1-Pin_8): track 0.00 -> 7.62 mm
- net Net-(J1-Pin_7): track 0.00 -> 7.62 mm
- net GPIO17: track 7.62 -> 14.1 mm
- net GPIO15: track 7.62 -> 14.1 mm
- net GPIO16: track 7.62 -> 14.1 mm
Other:
- board size 65.3 x 78.6 mm -> 65.3 x 78 mm
